Commit message: Refactor driver node and URDF: streamline comments, improve geometry definitions, and correct joint orientations for better accuracy in pan-tilt control.

File: urdf/pan_tilt.urdf (robot description, URDF)
Before this commit: robot pan_tilt_turret, 5 links, 4 joints
Joints:
- joint laser_joint: origin xyz=0.043 0 0 rpy=0 -1.5708 0 -> xyz=0.043 0 0 rpy=0 1.5708 0
- joint tilt_joint: origin xyz=0 0 0.075 rpy=0 0 0 -> xyz=0 0 0.075 rpy=0 -1.5708 0
